File: MP2303_tryout.kicad_pcb (KiCad board)
At the start: 2 copper layers, 12 parts, among them U1 MP2303A_ALT

Commit message: update,
Parts:
- L1: value L_10uH,CD74 -> L_10uH_shielded,CD127; footprint w_smd_inductors:inductor_smd_6x4.3mm -> footprint-lib:L_CD127_shielded
- U1: footprint Package_SO:SOIC-8_3.9x4.9mm_P1.27mm -> footprint-lib:MP2303,SOIC-8_3.9x4.9mm_P1.27mm,thermal_via
- moved L1 12.6 mm to (30.4, 48.0)
- moved U1 9.68 mm to (19.3, 36.3)
Connections:
- C2 pad 1: Net-(C2-Pad1) -> (no net)
